File: KiCAD/modular-development-board/modular-development-board.sch (KiCad schematic (older format))
At the start: 63 parts, among them J1 Power In, J10 DHT11-LEDS, J11 Buzzzer-Light, J12 USB_B_Micro, J13 UART, J2 5V Out, J3 3V3 Out, J4 GND, J5 Digital 1, J6 Digital 2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

Commit message: Added modular developmend board design and test software.
Parts:
- added J14: Power In, Connector_PinSocket_2.54mm:PinSocket_1x02_P2.54mm_Vertical, symbol Connector:Conn_01x02_Female
- F1: value 2A 24V PTC -> FSMD200-242920-R
- J12: footprint Connector_USB:USB_Micro-B_GCT_USB3076-30-A -> Footprints:KLS1-233-Micro-USB
Connections:
- wire segments 270 -> 274
Other:
- note added: "Hold Current = 2A\nTrip Current = 4A"
- note added: "TODO: 16MHz Osc \nError - 2 and 4 must \nbe GND (reverse them)."
- note added: "TODO: Add 1k to TX and RX line."
- note added: "TODO: Add TX \nand RX LEDs."
- note added: "TODO: Add VBUS to the 5V \nrail with schotky diode."
- note added: "TODO: Connect Buzzer\nto different pin."
- note added: "TODO: Connect LIGHT\nto Analog 0 pin.\nChange resistor position."
- note added: "TODO: Incorrect 2N2222\nin PCB."
- note added: "TODO: Increase Power \nLED resistor to 4.7k."
- note added: "Vf=0.35V"
- moved on the sheet: D1
